File: BML-Badges/_autosave-.kicad_pcb (KiCad board)
At the start: 2 copper layers, 19 parts, among them Q1 PN2222A, Q2 PN2222A, Q3 PN2222A

Commit message: Naptime
Parts:
- C1, C2, C3: footprint C2V8 -> C1V8
- Q1, Q2, Q3: footprint TO92-EBC-num -> TO92-CBE
- moved C1 360.5 mm to (0.00, 0.00)
- moved PHOTOR1 352.5 mm to (0.00, 0.00)
- moved C2 351.8 mm to (0.00, 0.00)
- moved D1 345.4 mm to (0.00, 0.00)
- moved PHOTOR2 343.6 mm to (0.00, 0.00)
- moved C3 343.3 mm to (0.00, 0.00)
- moved Q1 338.4 mm to (0.00, 0.00), turned to 0 degrees
- moved R1 335.8 mm to (0.00, 0.00), turned to 0 degrees
- moved D2 335.4 mm to (0.00, 0.00)
- moved PHOTOR3 334.9 mm to (0.00, 0.00)
- moved R2 334.7 mm to (0.00, 0.00)
- moved Q2 331.0 mm to (0.00, 0.00)
- moved D3 327.5 mm to (0.00, 0.00)
- moved R3 327.5 mm to (0.00, 0.00), turned to 0 degrees
- moved R4 325.1 mm to (0.00, 0.00)
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Connections:
- BT1 pad 2: N-000008 -> N-000005
- C1 pad 1: N-000002 -> N-000004
- C1 pad 2: N-000008 -> N-000005
- C2 pad 1: N-000009 (its old number) -> N-000003
- C2 pad 2: N-000008 -> N-000005
- C3 pad 1: N-000006 -> N-000008
- C3 pad 2: N-000008 -> N-000005
- D1 pad 2: N-000001 (its old number) -> N-000002
- D2 pad 2: N-000004 -> N-0000011
- D3 pad 2: N-000005 -> N-000006
- PHOTOR1 pad 1: N-000002 -> N-000004
- PHOTOR1 pad 2: N-000008 -> N-000005
- PHOTOR2 pad 1: N-000009 (its old number) -> N-000003
- PHOTOR2 pad 2: N-000008 -> N-000005
- PHOTOR3 pad 1: N-000006 -> N-000008
- PHOTOR3 pad 2: N-000008 -> N-000005
- R2 pad 2: N-000002 -> N-000004
- R4 pad 2: N-000009 (its old number) -> N-000003
- R6 pad 2: N-000006 -> N-000008
Other:
- rule pad_to_mask_clearance: 0 -> 0.2
