File: BML-Badges/BML-Badges.kicad_pcb (KiCad board)
At the start: 2 copper layers, 19 parts, among them Q1 PN2222A, Q2 PN2222A, Q3 PN2222A

Commit message: version1complete
Parts:
- BT1: moved to B.Cu
- moved Q2 31.0 mm to (238.8, 181.6), turned to 180 degrees
- moved R6 29.7 mm to (222.2, 182.9), turned to 180 degrees
- moved C3 29.0 mm to (227.3, 218.4)
- moved PHOTOR3 29.0 mm to (227.3, 205.7)
- moved D3 28.4 mm to (227.3, 195.6)
- moved Q1 28.2 mm to (251.5, 181.6), turned to 180 degrees
- moved Q3 28.2 mm to (229.9, 182.9)
- moved R2 27.8 mm to (247.0, 196.8), turned to 270 degrees
- moved C2 26.8 mm to (241.3, 218.4)
- moved PHOTOR2 26.8 mm to (241.3, 205.7)
- moved D1 26.2 mm to (252.7, 195.6)
- moved D2 26.2 mm to (240.0, 195.6)
- moved C1 25.7 mm to (254.0, 218.4)
- moved PHOTOR1 25.7 mm to (254.0, 205.7)
- moved R3 25.4 mm to (234.3, 192.4)
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Connections:
- BT1 pad 2: N-000008 -> GND
- C1 pad 1: N-000002 (its old number) -> N-000001
- C1 pad 2: N-000008 -> GND
- C2 pad 2: N-000008 -> GND
- C3 pad 2: N-000008 -> GND
- PHOTOR1 pad 1: N-000002 (its old number) -> N-000001
- PHOTOR1 pad 2: N-000008 -> GND
- PHOTOR2 pad 2: N-000008 -> GND
- PHOTOR3 pad 2: N-000008 -> GND
- Q1 pad 1: N-000008 -> (no net)
- Q1 pad 2: N-000002 (its old number) -> GND
- Q2 pad 1: N-000008 -> (no net)
- Q3 pad 1: N-000008 -> (no net)
- Q3 pad 2: N-000006 -> GND
- R2 pad 2: N-000002 (its old number) -> N-000001
Routing:
- net N-0000010: track 0.00 -> 76.9 mm
- net N-000009: track 0.00 -> 38.2 mm
- net N-000006: track 0.00 -> 37.1 mm
- net N-000001: track 0.00 -> 22.2 mm
- net N-000002: track 0.00 -> 18.6 mm
- net N-000004: track 0.00 -> 16.1 mm
- net N-000005: track 0.00 -> 13.5 mm
- net N-000003: track 0.00 -> 12.7 mm
- net N-000007: track 0.00 -> 6.35 mm
- net N-0000011: track 0.00 -> 5.23 mm
- added copper zone on F.Cu, net GND
Other:
- board outline added: 43.2 x 45.7 mm
- board text added: "Karmanya Aggarwal BML Munjal University"

Commit message: floating transistors
Connections:
- BT1 pad 1: N-0000010 (its old number) -> 3V
- Q1 pad 1: (no net) -> GND
- Q1 pad 2: GND -> N-000001
- Q2 pad 1: (no net) -> GND
- Q3 pad 1: (no net) -> GND
- Q3 pad 2: GND -> N-000006
- R1 pad 1: N-0000010 (its old number) -> 3V
- R2 pad 1: N-0000010 (its old number) -> 3V
- R3 pad 1: N-0000010 (its old number) -> 3V
- R4 pad 1: N-0000010 (its old number) -> 3V
- R5 pad 1: N-0000010 (its old number) -> 3V
- R6 pad 1: N-0000010 (its old number) -> 3V
Routing:
- net N-0000010 (its old number): track 76.9 -> 0.00 mm
- net 3V: track 0.00 -> 76.9 mm
- net N-000001: track 22.2 -> 46.6 mm
- net N-000006: track 37.1 -> 48.0 mm

Commit message: floating transistors
Routing:
- net GND: track 0.00 -> 6.88 mm
Changed lines of the file:
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@@
   (general
     (links 30)
-    (no_connects 1)
+    (no_connects 0)
     (area 218.389999 177.749999 267.439525 223.570001)
     (thickness 1.6)
     (drawings 5)
-    (tracks 58)
+    (tracks 60)
     (zones 0)
     (modules 19)
@@
   (segment (start 234.315 191.135) (end 235.585 191.135) (width 0.254) (layer B.Cu) (net 1))
   (segment (start 235.585 191.135) (end 237.49 189.23) (width 0.254) (layer B.Cu) (net 1))
+  (segment (start 231.14 181.61) (end 236.22 181.61) (width 0.254) (layer B.Cu) (net 2) (status 400000))
+  (segment (start 236.22 181.61) (end 237.49 182.88) (width 0.254) (layer B.Cu) (net 2) (status 800000))
   (segment (start 252.73 182.88) (end 252.73 189.23) (width 0.254) (layer B.Cu) (net 3) (status 400000))
   (segment (start 251.46 200.025) (end 251.46 205.74) (width 0.254) (layer B.Cu) (net 3) (status 800000))
