File: BML-Badges/BML-Badges.sch (KiCad schematic (older format))
At the start: 19 parts, among them Q1 PN2222A, Q2 PN2222A, Q3 PN2222A

Commit message: version1complete
Connections:
- net GND: now reaches BT1.2 (-), C1.2, C2.2, C3.2, PHOTOR1.2, PHOTOR2.2, PHOTOR3.2, Q1.1 (E), Q2.1 (E), Q3.1 (E)
Changed lines of the file:
@@
 Sheet 1 1
 Title "Analog Components Light Reactive LEDs"
-Date "20 aug 2015"
+Date "21 aug 2015"
 Rev "1"
 Comp "BML Munjal University"
@@
 	0    -1   -1   0
 $EndComp
+Text GLabel 6300 3050 0    60   Input ~ 0
+GND
+Wire Wire Line
+	6300 3050 6300 2900
+Connection ~ 6300 2900
 $EndSCHEMATC

Commit message: floating transistors
Connections:
- net 3V: now reaches BT1.1 (+), R1.1, R2.1, R3.1, R4.1, R5.1, R6.1
Changed lines of the file:
@@
 EESchema Schematic File Version 2
+LIBS:pn2222a
 LIBS:open-project
 LIBS:power
@@
 LIBS:contrib
 LIBS:valves
-LIBS:pn2222a
 LIBS:BML-Badges-cache
 EELAYER 27 0
@@
 Connection ~ 8400 1700
 Wire Wire Line
-	8950 1250 8950 2900
+	8950 2900 8950 1250
 Wire Wire Line
 	8950 1250 8600 1250
@@
 	3450 2350 6000 2350
 Wire Wire Line
-	8950 2900 5800 2900
+	5800 2900 8950 2900
 Wire Wire Line
 	6000 2900 6050 2900
@@
 	0    -1   -1   0
 $EndComp
+Text GLabel 6300 3050 0    60   Input ~ 0
+GND
+Wire Wire Line
+	6300 3050 6300 2900
+Connection ~ 6300 2900
+Text GLabel 4500 3050 0    60   Input ~ 0
+3V
+Wire Wire Line
+	4500 3050 4500 2900
+Connection ~ 4500 2900
+$Comp
+L PN2222A Q1
+U 1 1 55D6A256
+P 2900 1350
+F 0 "Q1" H 2900 1202 40  0000 R CNN
+F 1 "PN2222A" H 2900 1500 40  0000 R CNN
+F 2 "TO92" H 2800 1452 29  0000 C CNN
+F 3 "" H 2900 1350 60  0000 C CNN
+	1    2900 1350
+	0    -1   -1   0
+$EndComp
 $Comp
 L PN2222A Q2
-U 1 1 55D5E955
+U 1 1 55D6A272
 P 5450 1300
 F 0 "Q2" H 5450 1152 40  0000 R CNN
@@
 	0    -1   -1   0
 $EndComp
-$Comp
-L PN2222A Q1
-U 1 1 55D5E95B
-P 2900 1350
-F 0 "Q1" H 2900 1202 40  0000 R CNN
-F 1 "PN2222A" H 2900 1500 40  0000 R CNN
-F 2 "TO92" H 2800 1452 29  0000 C CNN
-F 3 "" H 2900 1350 60  0000 C CNN
-	1    2900 1350
-	0    -1   -1   0
-$EndComp
-Text GLabel 6300 3050 0    60   Input ~ 0
-GND
-Wire Wire Line
-	6300 3050 6300 2900
-Connection ~ 6300 2900
 $EndSCHEMATC

Commit message: Added Anools Contribution
Parts:
- C1, C2, C3: symbol C -> C-RESCUE-BML-Badges
- D1, D2, D3: symbol LED -> LED-RESCUE-BML-Badges
- R1, R3, R5: value 330 -> 50; symbol R -> R-RESCUE-BML-Badges
- R2, R4, R6: symbol R -> R-RESCUE-BML-Badges
Changed lines of the file:
@@
 EESchema Schematic File Version 2
+LIBS:BML-Badges-rescue
 LIBS:pn2222a
 LIBS:open-project
@@
 LIBS:memory
 LIBS:xilinx
-LIBS:special
 LIBS:microcontrollers
 LIBS:dsp
@@
 LIBS:valves
 LIBS:BML-Badges-cache
-EELAYER 27 0
+EELAYER 25 0
 EELAYER END
 $Descr A4 11693 8268
@@
 $EndDescr
 $Comp
-L LED D3
+L LED-RESCUE-BML-Badges D3
 U 1 1 55D5B114
 P 7850 1250
@@
 $EndComp
 $Comp
-L R R5
+L R-RESCUE-BML-Badges R5
 U 1 1 55D5B123
 P 7350 1250
 F 0 "R5" V 7430 1250 40  0000 C CNN
-F 1 "330" V 7357 1251 40  0000 C CNN
+F 1 "50" V 7357 1251 40  0000 C CNN
 F 2 "~" V 7280 1250 30  0000 C CNN
 F 3 "~" H 7350 1250 30  0000 C CNN
@@
 $EndComp
 $Comp
-L R R6
+L R-RESCUE-BML-Badges R6
 U 1 1 55D5B132
 P 8050 1700
@@
 $EndComp
 $Comp
-L C C3
+L C-RESCUE-BML-Badges C3
 U 1 1 55D5B141
 P 8750 2100
@@
 Connection ~ 8950 2100
 $Comp
-L LED D2
+L LED-RESCUE-BML-Badges D2
 U 1 1 55D5B7CB
 P 4900 1200
@@
 $EndComp
 $Comp
-L R R3
+L R-RESCUE-BML-Badges R3
 U 1 1 55D5B7D1
 P 4400 1200
 F 0 "R3" V 4480 1200 40  0000 C CNN
-F 1 "330" V 4407 1201 40  0000 C CNN
+F 1 "50" V 4407 1201 40  0000 C CNN
 F 2 "~" V 4330 1200 30  0000 C CNN
 F 3 "~" H 4400 1200 30  0000 C CNN
@@
 $EndComp
 $Comp
-L R R4
+L R-RESCUE-BML-Badges R4
 U 1 1 55D5B7D7
 P 5100 1650
@@
 $EndComp
 $Comp
-L C C2
+L C-RESCUE-BML-Badges C2
 U 1 1 55D5B7DD
 P 5800 2050
@@
 Connection ~ 6000 2050
 $Comp
-L LED D1
+L LED-RESCUE-BML-Badges D1
 U 1 1 55D5B7FC
 P 2350 1250
@@
 $EndComp
 $Comp
-L R R1
+L R-RESCUE-BML-Badges R1
 U 1 1 55D5B802
 P 1850 1250
 F 0 "R1" V 1930 1250 40  0000 C CNN
-F 1 "330" V 1857 1251 40  0000 C CNN
+F 1 "50" V 1857 1251 40  0000 C CNN
 F 2 "~" V 1780 1250 30  0000 C CNN
 F 3 "~" H 1850 1250 30  0000 C CNN
@@
 $EndComp
 $Comp
-L R R2
+L R-RESCUE-BML-Badges R2
 U 1 1 55D5B808
 P 2550 1700
@@
 $EndComp
 $Comp
-L C C1
+L C-RESCUE-BML-Badges C1
 U 1 1 55D5B80E
 P 3250 2100
