File: BML-Badges-anool/BML-Badges.sch (KiCad schematic (older format))
At the start: 19 parts, among them Q1 PN2222A, Q2 PN2222A, Q3 PN2222A

Commit message: Added Anools Contribution
Parts:
- added P1: +3V, BML-Badges:1pin, symbol CONN_01X01
- added P2: GND, BML-Badges:1pin, symbol CONN_01X01
- BT1: footprint ~ -> BML-Badges:BS-7-CR2032-2
- C1: footprint ~ -> BML-Badges:C2V8; symbol C -> C-RESCUE-BML-Badges
- C2, C3: footprint ~ -> BML-Badges:C2V8
- D1, D2, D3: footprint ~ -> BML-Badges:LED-5MM
- PHOTOR1, PHOTOR2, PHOTOR3: footprint ~ -> BML-Badges:LDR
- Q1, Q2, Q3: footprint TO92 -> BML-Badges:TO92-EBC-num
- R1, R2, R3, R4, R5, R6: footprint ~ -> BML-Badges:R1
Connections:
- net 3V: now also P1.1 (P1)
- net GND: now also P2.1 (P1)
Changed lines of the file:
@@
 EESchema Schematic File Version 2
-LIBS:pn2222a
-LIBS:open-project
+LIBS:bml-badges
+LIBS:BML-Badges-rescue
 LIBS:power
-LIBS:device
-LIBS:transistors
-LIBS:conn
-LIBS:linear
-LIBS:regul
-LIBS:74xx
-LIBS:cmos4000
-LIBS:adc-dac
-LIBS:memory
-LIBS:xilinx
-LIBS:special
-LIBS:microcontrollers
-LIBS:dsp
-LIBS:microchip
-LIBS:analog_switches
-LIBS:motorola
-LIBS:texas
-LIBS:intel
-LIBS:audio
-LIBS:interface
-LIBS:digital-audio
-LIBS:philips
-LIBS:display
-LIBS:cypress
-LIBS:siliconi
-LIBS:opto
-LIBS:atmel
-LIBS:contrib
-LIBS:valves
 LIBS:BML-Badges-cache
 EELAYER 27 0
@@
 F 0 "D3" H 7850 1350 50  0000 C CNN
 F 1 "LED" H 7850 1150 50  0000 C CNN
-F 2 "~" H 7850 1250 60  0000 C CNN
+F 2 "BML-Badges:LED-5MM" H 7850 1250 60  0001 C CNN
 F 3 "~" H 7850 1250 60  0000 C CNN
 	1    7850 1250
@@
 F 0 "R5" V 7430 1250 40  0000 C CNN
 F 1 "330" V 7357 1251 40  0000 C CNN
-F 2 "~" V 7280 1250 30  0000 C CNN
+F 2 "BML-Badges:R1" V 7280 1250 30  0001 C CNN
 F 3 "~" H 7350 1250 30  0000 C CNN
 	1    7350 1250
@@
 F 0 "R6" V 8130 1700 40  0000 C CNN
 F 1 "100k" V 8057 1701 40  0000 C CNN
-F 2 "~" V 7980 1700 30  0000 C CNN
+F 2 "BML-Badges:R1" V 7980 1700 30  0001 C CNN
 F 3 "~" H 8050 1700 30  0000 C CNN
 	1    8050 1700
@@
 F 0 "C3" H 8750 2200 40  0000 L CNN
 F 1 "22uF" H 8756 2015 40  0000 L CNN
-F 2 "~" H 8788 1950 30  0000 C CNN
+F 2 "BML-Badges:C2V8" H 8788 1950 30  0001 C CNN
 F 3 "~" H 8750 2100 60  0000 C CNN
 	1    8750 2100
@@
 F 0 "BT1" H 5500 3100 50  0000 C CNN
 F 1 "3V" H 5500 2710 50  0000 C CNN
-F 2 "~" H 5500 2900 60  0000 C CNN
+F 2 "BML-Badges:BS-7-CR2032-2" H 5500 2900 60  0001 C CNN
 F 3 "~" H 5500 2900 60  0000 C CNN
 	1    5500 2900
@@
 F 0 "PHOTOR3" V 8800 1650 50  0000 C CNN
 F 1 "PHOTOR" V 8700 1700 50  0000 C CNN
-F 2 "~" H 8700 1700 60  0000 C CNN
+F 2 "BML-Badges:LDR" H 8700 1700 60  0001 C CNN
 F 3 "~" H 8700 1700 60  0000 C CNN
 	1    8700 1700
@@
 F 0 "D2" H 4900 1300 50  0000 C CNN
 F 1 "LED" H 4900 1100 50  0000 C CNN
-F 2 "~" H 4900 1200 60  0000 C CNN
+F 2 "BML-Badges:LED-5MM" H 4900 1200 60  0001 C CNN
 F 3 "~" H 4900 1200 60  0000 C CNN
 	1    4900 1200
@@
 F 0 "R3" V 4480 1200 40  0000 C CNN
 F 1 "330" V 4407 1201 40  0000 C CNN
-F 2 "~" V 4330 1200 30  0000 C CNN
+F 2 "BML-Badges:R1" V 4330 1200 30  0001 C CNN
 F 3 "~" H 4400 1200 30  0000 C CNN
 	1    4400 1200
@@
 F 0 "R4" V 5180 1650 40  0000 C CNN
 F 1 "100k" V 5107 1651 40  0000 C CNN
-F 2 "~" V 5030 1650 30  0000 C CNN
+F 2 "BML-Badges:R1" V 5030 1650 30  0001 C CNN
 F 3 "~" H 5100 1650 30  0000 C CNN
 	1    5100 1650
@@
 F 0 "C2" H 5800 2150 40  0000 L CNN
 F 1 "22uF" H 5806 1965 40  0000 L CNN
-F 2 "~" H 5838 1900 30  0000 C CNN
+F 2 "BML-Badges:C2V8" H 5838 1900 30  0001 C CNN
 F 3 "~" H 5800 2050 60  0000 C CNN
 	1    5800 2050
@@
 F 0 "PHOTOR2" V 5850 1600 50  0000 C CNN
 F 1 "PHOTOR" V 5750 1650 50  0000 C CNN
-F 2 "~" H 5750 1650 60  0000 C CNN
+F 2 "BML-Badges:LDR" H 5750 1650 60  0001 C CNN
 F 3 "~" H 5750 1650 60  0000 C CNN
 	1    5750 1650
@@
 	5450 1500 5450 2050
 Connection ~ 5450 1650
-Wire Wire Line
-	6000 1200 6000 2900
 Wire Wire Line
 	6000 1200 5650 1200
@@
 F 0 "D1" H 2350 1350 50  0000 C CNN
 F 1 "LED" H 2350 1150 50  0000 C CNN
-F 2 "~" H 2350 1250 60  0000 C CNN
+F 2 "BML-Badges:LED-5MM" H 2350 1250 60  0001 C CNN
 F 3 "~" H 2350 1250 60  0000 C CNN
 	1    2350 1250
@@
 F 0 "R1" V 1930 1250 40  0000 C CNN
 F 1 "330" V 1857 1251 40  0000 C CNN
-F 2 "~" V 1780 1250 30  0000 C CNN
+F 2 "BML-Badges:R1" V 1780 1250 30  0001 C CNN
 F 3 "~" H 1850 1250 30  0000 C CNN
 	1    1850 1250
@@
 F 0 "R2" V 2630 1700 40  0000 C CNN
 F 1 "100k" V 2557 1701 40  0000 C CNN
-F 2 "~" V 2480 1700 30  0000 C CNN
+F 2 "BML-Badges:R1" V 2480 1700 30  0001 C CNN
 F 3 "~" H 2550 1700 30  0000 C CNN
 	1    2550 1700
@@
 $EndComp
 $Comp
-L C C1
+L C-RESCUE-BML-Badges C1
 U 1 1 55D5B80E
 P 3250 2100
 F 0 "C1" H 3250 2200 40  0000 L CNN
 F 1 "22uF" H 3256 2015 40  0000 L CNN
-F 2 "~" H 3288 1950 30  0000 C CNN
+F 2 "BML-Badges:C2V8" H 3288 1950 30  0001 C CNN
 F 3 "~" H 3250 2100 60  0000 C CNN
 	1    3250 2100
@@
 F 0 "PHOTOR1" V 3300 1650 50  0000 C CNN
 F 1 "PHOTOR" V 3200 1700 50  0000 C CNN
-F 2 "~" H 3200 1700 60  0000 C CNN
+F 2 "BML-Badges:LDR" H 3200 1700 60  0001 C CNN
 F 3 "~" H 3200 1700 60  0000 C CNN
 	1    3200 1700
@@
 	7100 2450 4900 2450
 Wire Wire Line
-	4900 2450 4900 2900
+	4900 2450 4900 3250
 Connection ~ 4900 2900
 Wire Wire Line
@@
 Wire Wire Line
 	5800 2900 8950 2900
-Wire Wire Line
-	6000 2900 6050 2900
-Connection ~ 6050 2900
-Connection ~ 6000 2350
 $Comp
 L PN2222A Q3
@@
 F 0 "Q3" H 8400 1202 40  0000 R CNN
 F 1 "PN2222A" H 8400 1500 40  0000 R CNN
-F 2 "TO92" H 8300 1452 29  0000 C CNN
+F 2 "BML-Badges:TO92-EBC-num" H 8300 1452 29  0001 C CNN
 F 3 "" H 8400 1350 60  0000 C CNN
 	1    8400 1350
 	0    -1   -1   0
 $EndComp
-Text GLabel 6300 3050 0    60   Input ~ 0
+Text GLabel 6300 3050 2    60   Input ~ 0
 GND
 Wire Wire Line
@@
 F 0 "Q1" H 2900 1202 40  0000 R CNN
 F 1 "PN2222A" H 2900 1500 40  0000 R CNN
-F 2 "TO92" H 2800 1452 29  0000 C CNN
+F 2 "BML-Badges:TO92-EBC-num" H 2800 1452 29  0001 C CNN
 F 3 "" H 2900 1350 60  0000 C CNN
 	1    2900 1350
@@
 F 0 "Q2" H 5450 1152 40  0000 R CNN
 F 1 "PN2222A" H 5450 1450 40  0000 R CNN
-F 2 "TO92" H 5350 1402 29  0000 C CNN
+F 2 "BML-Badges:TO92-EBC-num" H 5350 1402 29  0001 C CNN
 F 3 "" H 5450 1300 60  0000 C CNN
 	1    5450 1300
 	0    -1   -1   0
 $EndComp
+$Comp
+L CONN_01X01 P1
+U 1 1 55D6EE92
+P 4900 3450
+F 0 "P1" H 4900 3550 50  0000 C CNN
+F 1 "+3V" V 5000 3450 50  0000 C CNN
+F 2 "BML-Badges:1pin" H 4900 3450 60  0001 C CNN
+F 3 "" H 4900 3450 60  0000 C CNN
+	1    4900 3450
+	0    1    1    0
+$EndComp
+Wire Wire Line
+	6000 1200 6000 3250
+Connection ~ 6000 2900
+Connection ~ 6000 2350
+$Comp
+L CONN_01X01 P2
+U 1 1 55D6F15A
+P 6000 3450
+F 0 "P2" H 6000 3550 50  0000 C CNN
+F 1 "GND" V 6100 3450 50  0000 C CNN
+F 2 "BML-Badges:1pin" H 6000 3450 60  0001 C CNN
+F 3 "" H 6000 3450 60  0000 C CNN
+	1    6000 3450
+	0    1    1    0
+$EndComp
 $EndSCHEMATC
